Commit message: Changes to type of robot and nav2 stack

File: install/box_bot_description/share/box_bot_description/robot/box_bot.xacro (robot description, xacro)
@@ -1 +1,20 @@
-/home/swarmmaster/thesis_ws/src/box_bot/box_bot_description/robot/box_bot.xacro
+<?xml version="1.0" ?>
+<robot name="box_bot" xmlns:xacro="http://www.ros.org/wiki/xacro">
+  <xacro:include filename="$(find box_bot_description)/robot/materials.xacro" />
+  <xacro:include filename="$(find box_bot_description)/robot/properties.xacro" />
+  <xacro:include filename="$(find box_bot_description)/robot/macros.xacro" />
+  <xacro:include filename="$(find box_bot_description)/robot/wheels.xacro" />
+  <xacro:include filename="$(find box_bot_description)/robot/caster_wheels.xacro" />
+  <xacro:include filename="$(find box_bot_description)/robot/box_bot_body.xacro" />
+  <xacro:include filename="$(find box_bot_description)/robot/box_bot.gazebo" />
+  <!--
+  <xacro:include filename="$(find box_bot_description)/robot/box_bot_propeller.xacro" />
+  -->
+  <xacro:box_bot_body parent_name="${base_name}"/>
+  <xacro:link_wheel name="right_wheel" r="${wheel_radius}" l="${wheel_width}" incr="${wheel_increment}"/>
+  <xacro:joint_wheel name="joint_right_wheel" parent="${base_name}" child="right_wheel" origin_xyz="0 ${base_box_x / 2.0} ${-1.0 * wheel_radius}" />
+  <xacro:link_wheel name="left_wheel" r="${wheel_radius}" l="${wheel_width}" incr="${wheel_increment}"/>
+  <xacro:joint_wheel name="joint_left_wheel" parent="${base_name}" child="left_wheel" origin_xyz="0 ${-1.0 * base_box_x / 2.0} ${-1.0 * wheel_radius}" />
+  <xacro:caster_wheel parent="chassis" caster_wheel_name="front" origin_xyz="${(base_box_x / 2.0) - wheel_increment} 0 ${-1.0* base_box_x / 2.0}" radius="${wheel_increment}" legth="${dummy_length}"/>
+  <xacro:caster_wheel parent="chassis" caster_wheel_name="back" origin_xyz="${(-1.0 *base_box_x / 2.0) + wheel_increment} 0 ${-1.0* base_box_x / 2.0}" radius="${wheel_increment}" legth="${dummy_length}"/>
+</robot>

File: install/box_bot_description/share/box_bot_description/robot/box_bot_body.xacro (robot description, xacro)
@@ -1 +1,36 @@
-/home/swarmmaster/thesis_ws/src/box_bot/box_bot_description/robot/box_bot_body.xacro
+<?xml version="1.0"?>
+<robot xmlns:xacro="http://www.ros.org/wiki/xacro">
+    <xacro:macro  name="box_bot_body" params="parent_name">
+      <link name="base_link">
+      </link>
+      <link name="${parent_name}">
+        <!-- pose and inertial -->
+        <pose>0 0 0 0 0 0</pose>
+        <inertial>
+          <mass value="${base_box_mass}"/>
+          <origin rpy="0 0 0" xyz="0 0 0"/>
+          <xacro:box_inertia mass="0.2" x="${base_box_x}" y="${base_box_y}" z="${base_box_z}"/>
+          <inertia ixx="0.000241935" ixy="0" ixz="0" iyy="0.000241935" iyz="0" izz="0.000241935"/>
+        </inertial>
+        <!-- body -->
+        <collision name="collision_${parent_name}">
+          <geometry>
+            <box size="${base_box_x} ${base_box_y} ${base_box_z}"/>
+          </geometry>
+        </collision>
+        <visual name="visual_${parent_name}">
+          <geometry>
+            <box size="${base_box_x} ${base_box_y} ${base_box_z}"/>
+          </geometry>
+        </visual>
+      </link>
+      <gazebo reference="chassis">
+        <material>Gazebo/Red</material>
+      </gazebo>
+      <joint name="base_link_joint" type="fixed">
+        <origin rpy="0 0 0" xyz="0 0 0" />
+        <parent link="base_link" />
+        <child link="${parent_name}" />
+      </joint>
+    </xacro:macro >
+</robot>

File: install/box_bot_description/share/box_bot_description/robot/box_bot_propeller.xacro (robot description, xacro)
@@ -1 +1,42 @@
-/home/swarmmaster/thesis_ws/src/box_bot/box_bot_description/robot/box_bot_propeller.xacro
+<?xml version="1.0"?>
+<robot xmlns:xacro="http://www.ros.org/wiki/xacro">
+    <xacro:macro  name="box_bot_propeller" params="name parent incr origin_xyz origin_rpy">
+      <!-- PROELLER -->
+      <link name="${name}_propeller_top">
+        <inertial>
+          <mass value="0.2"/>
+          <origin rpy="0 1.5707 1.5707" xyz="0 0 0"/>
+            <xacro:cylinder_inertia mass="0.2" r="${r}" l="${l}" />
+        </inertial>
+        <collision name="link_right_wheel_collision">
+          <origin rpy="0 1.5707 1.5707" xyz="0 0 0"/>
+          <geometry>
+            <cylinder length="${l}" radius="${r + incr}"/>
+          </geometry>
+        </collision>
+        <visual>
+          <origin rpy="0 0 0" xyz="0 0.0 0.0" />
+          <geometry>
+            <mesh filename="package://box_bot_description/meshes/prop.stl" scale="1.0 1.0 1.0"/>
+          </geometry>
+        </visual>
+      </link>
+      <joint name="top_propeller_joint" type="continuous">
+        <origin rpy="0 0 0" xyz="0.0 0.0 0.0" />
+        <parent link="${parent}" />
+        <child link="${name}_propeller_top" />
+        <axis xyz="0 1 0" />
+        <limit effort="1000.0" velocity="100.0" />
+      </joint>
+    <transmission name="top_propeller_joint_trans">
+      <type>transmission_interface/SimpleTransmission</type>
+      <joint name="top_propeller_joint">
+        <hardwareInterface>EffortJointInterface</hardwareInterface>
+      </joint>
+      <actuator name="top_propeller_jointMotor">
+        <hardwareInterface>EffortJointInterface</hardwareInterface>
+        <mechanicalReduction>1</mechanicalReduction>
+      </actuator>
+    </transmission>
+    </xacro:macro >
+</robot>

File: install/box_bot_description/share/box_bot_description/robot/caster_wheels.xacro (robot description, xacro)
@@ -1 +1,113 @@
-/home/swarmmaster/thesis_ws/src/box_bot/box_bot_description/robot/caster_wheels.xacro
+<?xml version="1.0"?>
+<robot xmlns:xacro="http://www.ros.org/wiki/xacro">
+    <!-- Caster Wheels-->
+    <xacro:macro  name="caster_wheel" params="parent caster_wheel_name origin_xyz radius legth">
+      <!-- CASTER FRONT-->
+      <link name="${caster_wheel_name}_yaw_link">
+        <inertial>
+            <mass value="0.001"/>
+            <origin rpy="0 1.5707 1.5707" xyz="0 0 0"/>
+            <xacro:cylinder_inertia mass="0.001" r="${0.9 * radius/2.0}" l="${legth}" />
+          </inertial>
+          <collision name="link_right_wheel_collision">
+            <origin rpy="0 1.5707 1.5707" xyz="0 0 0"/>
+            <geometry>
+              <cylinder length="${legth}" radius="${0.9 * radius/2.0}"/>
+            </geometry>
+          </collision>
+      </link>
+      <joint name="${caster_wheel_name}_yaw_joint" type="continuous">
+        <origin rpy="0 0 0" xyz="${origin_xyz}" />
+        <parent link="${parent}" />
+        <child link="${caster_wheel_name}_yaw_link" />
+        <axis xyz="0 0 1" />
+        <limit effort="1000.0" velocity="100.0" />
+        <dynamics damping="0.0" friction="0.1"/>
+      </joint>
+      <transmission name="${caster_wheel_name}_yaw_joint_trans">
+      <type>transmission_interface/SimpleTransmission</type>
+      <joint name="${caster_wheel_name}_yaw_joint">
+        <hardwareInterface>EffortJointInterface</hardwareInterface>
+      </joint>
+      <actuator name="${caster_wheel_name}_yaw_jointMotor">
+        <hardwareInterface>EffortJointInterface</hardwareInterface>
+        <mechanicalReduction>1</mechanicalReduction>
+      </actuator>
+    </transmission>
+    <link name="${caster_wheel_name}_roll_link">
+        <inertial>
+            <mass value="0.001"/>
+            <origin rpy="0 1.5707 1.5707" xyz="0 0 0"/>
+            <xacro:cylinder_inertia mass="0.001" r="${0.9 * radius/2.0}" l="${legth}" />
+          </inertial>
+          <collision name="link_right_wheel_collision">
+            <origin rpy="0 1.5707 1.5707" xyz="0 0 0"/>
+            <geometry>
+              <cylinder length="${legth}" radius="${0.9 * radius/2.0}"/>
+            </geometry>
+          </collision>
+      </link>
+      <joint name="${caster_wheel_name}_roll_joint" type="continuous">
+        <origin rpy="0 0 0" xyz="0 0 0" />
+        <parent link="${caster_wheel_name}_yaw_link" />
+        <child link="${caster_wheel_name}_roll_link" />
+        <axis xyz="1 0 0" />
+        <limit effort="1000.0" velocity="100.0" />
+        <dynamics damping="0.0" friction="0.1"/>
+      </joint>
+      <transmission name="${caster_wheel_name}_roll_joint_trans">
+      <type>transmission_interface/SimpleTransmission</type>
+      <joint name="${caster_wheel_name}_roll_joint">
+        <hardwareInterface>EffortJointInterface</hardwareInterface>
+      </joint>
+      <actuator name="${caster_wheel_name}_roll_jointMotor">
+        <hardwareInterface>EffortJointInterface</hardwareInterface>
+        <mechanicalReduction>1</mechanicalReduction>
+      </actuator>
+    </transmission>
+      <link name="${caster_wheel_name}_pitch_link">
+        <inertial>
+          <mass value="0.001"/>
+          <origin rpy="0 1.5707 1.5707" xyz="0 0 0"/>
+            <xacro:sphere_inertia mass="0.001" r="${radius}"/>
+        </inertial>
+        <collision name="${caster_wheel_name}_collision">
+          <origin rpy="0 1.5707 1.5707" xyz="0 0 0"/>
+          <geometry>
+            <sphere radius="${radius}"/>
+          </geometry>
+        </collision>
+        <visual name="${caster_wheel_name}_visual">
+          <origin rpy="0 1.5707 1.5707" xyz="0 0 0"/>
+          <geometry>
+            <sphere radius="${radius}"/>
+          </geometry>
+        </visual>
+      </link>
+      <joint name="${caster_wheel_name}_pitch_joint" type="continuous">
+        <origin rpy="0 0 0" xyz="0 0 0" />
+        <parent link="${caster_wheel_name}_roll_link" />
+        <child link="${caster_wheel_name}_pitch_link" />
+        <axis xyz="0 1 0" />
+        <limit effort="1000.0" velocity="100.0" />
+        <dynamics damping="0.0" friction="0.1"/>
+      </joint>
+    <transmission name="${caster_wheel_name}_pitch_joint_trans">
+      <type>transmission_interface/SimpleTransmission</type>
+      <joint name="${caster_wheel_name}_pitch_joint">
+        <hardwareInterface>EffortJointInterface</hardwareInterface>
+      </joint>
+      <actuator name="${caster_wheel_name}_pitch_jointMotor">
+        <hardwareInterface>EffortJointInterface</hardwareInterface>
+        <mechanicalReduction>1</mechanicalReduction>
+      </actuator>
+    </transmission>
+    <gazebo reference="${caster_wheel_name}_pitch_link">
+      <kp>1000000000000000000000000000.0</kp>
+      <kd>1000000000000000000000000000.0</kd>
+      <mu1>${mu1_wheel}</mu1>
+      <mu2>${mu2_wheel}</mu2>
+      <material>Gazebo/Green</material>
+    </gazebo>
+  </xacro:macro >
+</robot>

File: install/box_bot_description/share/box_bot_description/robot/macros.xacro (robot description, xacro)
@@ -1 +1,21 @@
-/home/swarmmaster/thesis_ws/src/box_bot/box_bot_description/robot/macros.xacro
+<?xml version="1.0"?>
+<robot xmlns:xacro="http://www.ros.org/wiki/xacro">
+    <xacro:macro  name="cylinder_inertia" params="mass r l">
+      <inertia  ixx="${mass*(3*r*r+l*l)/12}" ixy = "0" ixz = "0"
+                iyy="${mass*(3*r*r+l*l)/12}" iyz = "0"
+                izz="${mass*(r*r)/2}" />
+    </xacro:macro >
+    <xacro:macro name="box_inertia" params="mass x y z">
+      <inertia  ixx="${mass*(y*y+z*z)/12}" ixy = "0" ixz = "0"
+                iyy="${mass*(x*x+z*z)/12}" iyz = "0"
+                izz="${mass*(x*x+z*z)/12}"
+      />
+    </xacro:macro>
+  <xacro:macro name="sphere_inertia" params="mass r">
+    <inertia
+          ixx="${2*mass*r*r/5}" ixy = "0" ixz = "0"
+          iyy="${2*mass*r*r/5}" iyz = "0"
+          izz="${2*mass*r*r/5}"
+    />
+  </xacro:macro>
+</robot>

File: install/box_bot_description/share/box_bot_description/robot/materials.xacro (robot description, xacro)
@@ -1 +1,27 @@
-/home/swarmmaster/thesis_ws/src/box_bot/box_bot_description/robot/materials.xacro
+<?xml version="1.0" ?>
+<robot>
+  <material name="black">
+    <color rgba="0.0 0.0 0.0 1.0"/>
+  </material>
+  <material name="blue">
+    <color rgba="0.203125 0.23828125 0.28515625 1.0"/>
+  </material>
+  <material name="green">
+    <color rgba="0.0 0.8 0.0 1.0"/>
+  </material>
+  <material name="grey">
+    <color rgba="0.2 0.2 0.2 1.0"/>
+  </material>
+  <material name="orange">
+    <color rgba="1.0 0.423529411765 0.0392156862745 1.0"/>
+  </material>
+  <material name="brown">
+    <color rgba="0.870588235294 0.811764705882 0.764705882353 1.0"/>
+  </material>
+  <material name="red">
+    <color rgba="0.80078125 0.12890625 0.1328125 1.0"/>
+  </material>
+  <material name="white">
+    <color rgba="1.0 1.0 1.0 1.0"/>
+  </material>
+</robot>

File: install/box_bot_description/share/box_bot_description/robot/properties.xacro (robot description, xacro)
@@ -1 +1,21 @@
-/home/swarmmaster/thesis_ws/src/box_bot/box_bot_description/robot/properties.xacro
+<?xml version="1.0"?>
+<robot xmlns:xacro="http://www.ros.org/wiki/xacro">
+	<!-- Constants -->
+	<xacro:property name="PI" value="3.1415926535897931"/>
+	<!-- Base Box -->
+    <xacro:property name="base_name" value="chassis"/>
+    <xacro:property name="base_box_mass" value="1.0"/>
+	<xacro:property name="base_box_x" value="0.1"/>
+    <xacro:property name="base_box_y" value="0.1"/>
+    <xacro:property name="base_box_z" value="0.1"/>
+    <!-- Wheels -->
+	<xacro:property name="wheel_radius" value="${base_box_z / 4.0}"/>
+    <xacro:property name="wheel_width" value="0.001"/>
+    <xacro:property name="wheel_increment" value="0.010"/>
+    <xacro:property name="mu1_wheel" value="0.5"/>
+    <xacro:property name="mu2_wheel" value="0.5"/>
+    <xacro:property name="kp_wheel" value="1000.0"/>
+    <xacro:property name="kd_wheel" value="1000.0"/>
+    <!--Caster Wheels-->
+    <xacro:property name="dummy_length" value="0.001"/>
+</robot>

File: install/box_bot_description/share/box_bot_description/robot/wheels.xacro (robot description, xacro)
@@ -1 +1,35 @@
-/home/swarmmaster/thesis_ws/src/box_bot/box_bot_description/robot/wheels.xacro
+<?xml version="1.0"?>
+<robot xmlns:xacro="http://www.ros.org/wiki/xacro">
+    <!-- Wheels-->
+    <xacro:macro  name="link_wheel" params="name r l incr">
+      <link name="${name}">
+          <inertial>
+            <mass value="0.2"/>
+            <origin rpy="0 1.5707 1.5707" xyz="0 0 0"/>
+              <xacro:cylinder_inertia mass="0.2" r="${r}" l="${l}" />
+          </inertial>
+          <collision name="link_right_wheel_collision">
+            <origin rpy="0 1.5707 1.5707" xyz="0 0 0"/>
+            <geometry>
+              <cylinder length="${l}" radius="${r + incr}"/>
+            </geometry>
+          </collision>
+          <visual name="link_right_wheel_visual">
+            <origin rpy="0 1.5707 1.5707" xyz="0 0 0"/>
+            <geometry>
+              <cylinder length="${l}" radius="${r + incr}"/>
+            </geometry>
+          </visual>
+      </link>
+  </xacro:macro >
+  <xacro:macro  name="joint_wheel" params="name parent child origin_xyz">
+    <joint name="${name}" type="continuous">
+      <origin rpy="0 0 0" xyz="${origin_xyz}"/>
+      <child link="${child}"/>
+      <parent link="${parent}"/>
+      <axis rpy="0 0 0" xyz="0 1 0"/>
+      <limit effort="10000" velocity="1000"/>
+      <joint_properties damping="1.0" friction="1.0"/>
+    </joint>
+  </xacro:macro >
+</robot>

File: install/linorobot2_description/share/linorobot2_description/urdf/2wd_properties.urdf.xacro (robot description, xacro)
@@ -1 +1,22 @@
-/home/swarmmaster/thesis_ws/src/linorobot2/linorobot2_description/urdf/2wd_properties.urdf.xacro
+<?xml version="1.0"?>
+<robot xmlns:xacro="http://ros.org/wiki/xacro">
+  <xacro:property name="base_length" value="0.24" />
+  <xacro:property name="base_width" value="0.275" />
+  <xacro:property name="base_height" value="0.003" />
+  <xacro:property name="base_mass" value="1" />
+  <xacro:property name="wheel_radius" value="0.045" />
+  <xacro:property name="wheel_width" value="0.01" />
+  <xacro:property name="wheel_pos_x" value="0.0" />
+  <xacro:property name="wheel_pos_y" value="0.13" />
+  <xacro:property name="wheel_pos_z" value="-0.03" />
+  <xacro:property name="wheel_mass" value=".1" />
+  <xacro:property name="wheel_torque" value="20" />
+  <xacro:property name="front_caster_wheel" value="true" />
+  <xacro:property name="rear_caster_wheel" value="true" />
+  <xacro:property name="laser_pose">
+    <origin xyz="0.12 0 0.33" rpy="0 0 0"/>
+  </xacro:property>
+  <xacro:property name="depth_sensor_pose">
+    <origin xyz="0.14 0.0 0.045" rpy="0 0 0"/>
+  </xacro:property>
+</robot>

File: install/linorobot2_description/share/linorobot2_description/urdf/4wd_properties.urdf.xacro (robot description, xacro)
@@ -1 +1,20 @@
-/home/swarmmaster/thesis_ws/src/linorobot2/linorobot2_description/urdf/4wd_properties.urdf.xacro
+<?xml version="1.0"?>
+<robot xmlns:xacro="http://ros.org/wiki/xacro">
+  <xacro:property name="base_length" value="0.445" />
+  <xacro:property name="base_width" value="0.200" />
+  <xacro:property name="base_height" value="0.129" />
+  <xacro:property name="base_mass" value="10" />
+  <xacro:property name="wheel_radius" value="0.07162" />
+  <xacro:property name="wheel_width" value="0.05" />
+  <xacro:property name="wheel_pos_x" value="0.120" />
+  <xacro:property name="wheel_pos_y" value="0.1355" />
+  <xacro:property name="wheel_pos_z" value="-0.04788" />
+  <xacro:property name="wheel_mass" value=".6" />
+  <xacro:property name="wheel_torque" value="20" />
+  <xacro:property name="laser_pose">
+    <origin xyz="-0.0475 0 0.125" rpy="0 0 0"/>
+  </xacro:property>
+  <xacro:property name="depth_sensor_pose">
+    <origin xyz="-0.065 0 0.255" rpy="0 0 0"/>
+  </xacro:property>
+</robot>

File: install/linorobot2_description/share/linorobot2_description/urdf/controllers/diff_drive.urdf.xacro (robot description, xacro)
@@ -1 +1,22 @@
-/home/swarmmaster/thesis_ws/src/linorobot2/linorobot2_description/urdf/controllers/diff_drive.urdf.xacro
+<robot xmlns:xacro="http://ros.org/wiki/xacro">
+  <xacro:macro name="diff_drive_controller" params="wheel_separation wheel_radius wheel_torque">
+    <gazebo>
+      <plugin name="differential_drive_controller" filename="libgazebo_ros_diff_drive.so">
+        <ros>
+          <argument>odom:=odom/unfiltered</argument>
+        </ros>
+        <updateRate>100</updateRate>
+        <left_joint>left_wheel_joint</left_joint>
+        <right_joint>right_wheel_joint</right_joint>
+        <wheel_separation>${wheel_separation}</wheel_separation>
+        <wheel_diameter>${wheel_radius * 2}</wheel_diameter>
+        <max_wheel_acceleration>1.0</max_wheel_acceleration>
+        <robot_base_frame>base_footprint</robot_base_frame>
+        <publish_odom>true</publish_odom>
+        <publish_odom_tf>false</publish_odom_tf>
+        <publish_wheel_tf>true</publish_wheel_tf>
+        <odometry_frame>odom</odometry_frame>
+      </plugin>
+    </gazebo>
+  </xacro:macro>
+</robot>

File: install/linorobot2_description/share/linorobot2_description/urdf/controllers/omni_drive.urdf.xacro (robot description, xacro)
@@ -1 +1,18 @@
-/home/swarmmaster/thesis_ws/src/linorobot2/linorobot2_description/urdf/controllers/omni_drive.urdf.xacro
+<robot xmlns:xacro="http://ros.org/wiki/xacro">
+  <xacro:macro name="omni_drive_controller">
+    <gazebo>
+    <plugin name="object_controller" filename="libgazebo_ros_planar_move.so">
+      <ros>
+        <argument>odom:=odom/unfiltered</argument>
+      </ros>
+      <command_topic>cmd_vel</command_topic>
+      <odometry_topic>odom/unfiltered</odometry_topic>
+      <odometry_frame>odom</odometry_frame>
+      <odometry_rate>20.0</odometry_rate>
+      <robot_base_frame>base_footprint</robot_base_frame>
+      <publish_odom>true</publish_odom>
+      <publish_odom_tf>false</publish_odom_tf>
+    </plugin>
+  </gazebo>
+  </xacro:macro>
+</robot>

File: install/linorobot2_description/share/linorobot2_description/urdf/controllers/skid_steer.urdf.xacro (robot description, xacro)
@@ -1 +1,27 @@
-/home/swarmmaster/thesis_ws/src/linorobot2/linorobot2_description/urdf/controllers/skid_steer.urdf.xacro
+<robot xmlns:xacro="http://ros.org/wiki/xacro">
+  <xacro:macro name="diff_drive_controller" params="wheel_separation wheel_radius wheel_torque">
+    <gazebo>
+      <plugin name="differential_drive_controller" filename="libgazebo_ros_diff_drive.so">
+        <ros>
+          <argument>odom:=odom/unfiltered</argument>
+        </ros>
+        <num_wheel_pairs>2</num_wheel_pairs>
+        <left_joint>front_left_wheel_joint</left_joint>
+        <right_joint>front_right_wheel_joint</right_joint>
+        <left_joint>rear_left_wheel_joint</left_joint>
+        <right_joint>rear_right_wheel_joint</right_joint>
+        <wheel_separation>${wheel_separation}</wheel_separation>
+        <wheel_separation>${wheel_separation}</wheel_separation>
+        <wheel_diameter>${wheel_radius * 2}</wheel_diameter>
+        <wheel_diameter>${wheel_radius * 2}</wheel_diameter>
+        <updateRate>100</updateRate>
+        <max_wheel_acceleration>1.0</max_wheel_acceleration>
+        <robot_base_frame>base_footprint</robot_base_frame>
+        <publish_odom>true</publish_odom>
+        <publish_odom_tf>false</publish_odom_tf>
+        <publish_wheel_tf>true</publish_wheel_tf>
+        <odometry_frame>odom</odometry_frame>
+      </plugin>
+    </gazebo>
+  </xacro:macro>
+</robot>

File: install/linorobot2_description/share/linorobot2_description/urdf/mecanum_properties.urdf.xacro (robot description, xacro)
@@ -1 +1,20 @@
-/home/swarmmaster/thesis_ws/src/linorobot2/linorobot2_description/urdf/mecanum_properties.urdf.xacro
+<?xml version="1.0"?>
+<robot xmlns:xacro="http://ros.org/wiki/xacro">
+  <xacro:property name="base_length" value="0.445" />
+  <xacro:property name="base_width" value="0.200" />
+  <xacro:property name="base_height" value="0.129" />
+  <xacro:property name="base_mass" value="10" />
+  <xacro:property name="wheel_radius" value="0.07162" />
+  <xacro:property name="wheel_width" value="0.05" />
+  <xacro:property name="wheel_pos_x" value="0.120" />
+  <xacro:property name="wheel_pos_y" value="0.1355" />
+  <xacro:property name="wheel_pos_z" value="-0.04788" />
+  <xacro:property name="wheel_mass" value=".6" />
+  <xacro:property name="wheel_torque" value="20" />
+  <xacro:property name="laser_pose">
+    <origin xyz="-0.0475 0 0.125" rpy="0 0 0"/>
+  </xacro:property>
+  <xacro:property name="depth_sensor_pose">
+    <origin xyz="0.2375 0 0.06" rpy="0 0 0"/>
+  </xacro:property>
+</robot>
