Commit message: Changes to type of robot and nav2 stack

File: install/linorobot2_description/share/linorobot2_description/urdf/mech/base.urdf.xacro (robot description, xacro)
@@ -1 +1,46 @@
-/home/swarmmaster/thesis_ws/src/linorobot2/linorobot2_description/urdf/mech/base.urdf.xacro
+<?xml version="1.0"?>
+<robot xmlns:xacro="http://ros.org/wiki/xacro">
+  <xacro:macro name="base" params="length width height mass wheel_radius wheel_pos_z">
+    <link name="base_footprint"/>
+    <link name="base_link">
+      <visual>
+        <origin xyz="0 0 0" rpy="0 0 0"/>
+        <geometry>
+          <box size="${length} ${width} ${height}"/>
+          <!-- <mesh filename="" scale="0.001 0.001 0.001"/> -->
+        </geometry>
+        <material name="yellow">
+          <color rgba="0.8784 0.6627 0.6627 1.0"/>
+        </material>
+      </visual>
+      <collision>
+        <origin xyz="0 0 0" rpy="0 0 0"/>
+        <geometry>
+          <box size="${length} ${width} ${height}"/>
+        </geometry>
+      </collision>
+      <inertial>
+        <origin xyz="0 0 0" rpy="0 0 0"/>
+        <mass value="${mass}"/>
+        <inertia ixx="${(1/12) * mass * ((width  * width)  + (height * height))}" ixy="0.0" ixz="0.0"
+                 iyy="${(1/12) * mass * ((length * length) + (height * height))}" iyz="0.0"
+                 izz="${(1/12) * mass * ((length * length) + (width  * width))}"/>
+      </inertial>
+    </link>
+    <gazebo reference="base_link">
+      <visual>
+        <material>
+          <ambient>0.8392 0.6314 0.0 1.0</ambient>
+          <diffuse>0.8392 0.6314 0.0 1.0</diffuse>
+          <specular>0.99 0.99 0.99 1.0</specular>
+          <emissive>0.0 0.0 0.0 0.0</emissive>
+        </material>
+      </visual>
+    </gazebo>
+    <joint name="base_to_footprint" type="fixed">
+      <parent link="base_footprint"/>
+      <child link="base_link"/>
+      <origin xyz="0 0 ${wheel_radius - wheel_pos_z}" rpy="0 0 0"/>
+    </joint>
+  </xacro:macro>
+</robot>

File: install/linorobot2_description/share/linorobot2_description/urdf/mech/caster_wheel.urdf.xacro (robot description, xacro)
@@ -1 +1,45 @@
-/home/swarmmaster/thesis_ws/src/linorobot2/linorobot2_description/urdf/mech/caster_wheel.urdf.xacro
+<?xml version="1.0"?>
+<robot xmlns:xacro="http://ros.org/wiki/xacro">
+  <xacro:macro name="caster_wheel" params="side mass base_length wheel_radius wheel_pos_z">
+    <xacro:property name="caster_wheel_radius" value="${(wheel_radius - wheel_pos_z) / 2}" />
+    <xacro:if value="${side == 'front'}">
+        <xacro:property name="caster_wheel_x" value="${(base_length / 2) - caster_wheel_radius}" />
+    </xacro:if>
+    <xacro:if value="${side == 'rear'}">
+        <xacro:property name="caster_wheel_x" value="${-(base_length / 2) + caster_wheel_radius}" />
+    </xacro:if>
+    <link name="${side}_caster_wheel_link">
+      <visual>
+        <origin xyz="0 0 0" rpy="0 0 0"/>
+        <geometry>
+          <sphere radius="${caster_wheel_radius}" />
+        </geometry>
+        <material name="black">
+            <color rgba="0.0 0.0 0.0 1.0"/>
+        </material>
+      </visual>
+      <collision>
+        <origin xyz="0 0 0" rpy="0 0 0"/>
+        <geometry>
+          <sphere radius="${caster_wheel_radius}" />
+        </geometry>
+      </collision>
+      <inertial>
+        <origin xyz="0 0 0" rpy="0 0 0"/>
+        <mass value="${mass}"/>
+        <inertia ixx="${(2/5) * mass * (caster_wheel_radius * caster_wheel_radius)}" ixy="0" ixz="0"
+                 iyy="${(2/5) * mass * (caster_wheel_radius * caster_wheel_radius)}" iyz="0"
+                 izz="${(2/5) * mass * (caster_wheel_radius * caster_wheel_radius)}" />
+      </inertial>
+    </link>
+    <gazebo reference="${side}_caster_wheel_link">
+        <mu1>0.01</mu1>
+        <mu2>0.01</mu2>
+    </gazebo>
+    <joint name="${side}_caster_wheel_joint" type="fixed">
+      <parent link="base_link"/>
+      <child link="${side}_caster_wheel_link"/>
+      <origin xyz="${caster_wheel_x} 0 -${caster_wheel_radius}" rpy="0 0 0"/>
+    </joint>
+  </xacro:macro>
+</robot>

File: install/linorobot2_description/share/linorobot2_description/urdf/mech/mecanum_wheel.urdf.xacro (robot description, xacro)
@@ -1 +1,49 @@
-/home/swarmmaster/thesis_ws/src/linorobot2/linorobot2_description/urdf/mech/mecanum_wheel.urdf.xacro
+<?xml version="1.0"?>
+<robot xmlns:xacro="http://ros.org/wiki/xacro">
+  <xacro:macro name="mecanum_wheel" params="side radius width pos_x pos_y pos_z mass">
+    <link name="${side}_wheel_link">
+      <visual>
+        <origin xyz="0 0 0" rpy="${pi/2} 0 0"/>
+        <geometry>
+          <cylinder radius="${radius}" length="${width}"/>
+        </geometry>
+        <material name="blue">
+            <color rgba="0.1764 0.4588 0.8509 1.0"/>
+        </material>
+      </visual>
+      <collision>
+        <origin xyz="0 0 0" rpy="${pi/2} 0 0"/>
+        <geometry>
+          <cylinder radius="${radius}" length="${width}"/>
+        </geometry>
+      </collision>
+      <inertial>
+        <origin xyz="0 0 0" rpy="0 0 0"/>
+        <mass value="${mass}"/>
+        <inertia ixx="${(2/5) * mass * (radius * radius)}" ixy="0" ixz="0"
+                 iyy="${(2/5) * mass * (radius * radius)}" iyz="0"
+                 izz="${(2/5) * mass * (radius * radius)}" />
+      </inertial>
+    </link>
+    <gazebo reference="${side}_wheel_link">
+        <mu1>0.01</mu1>
+        <mu2>0.01</mu2>
+    </gazebo>
+    <gazebo reference="${side}_wheel_link">
+      <visual>
+        <material>
+          <ambient>0.1764 0.4588 0.8509 1.0</ambient>
+          <diffuse>0.1764 0.4588 0.8509 1.0</diffuse>
+          <specular>0.1764 0.4588 0.8509 1.0</specular>
+          <emissive>0.0 0.0 0.0 0.0</emissive>
+        </material>
+      </visual>
+    </gazebo>
+    <joint name="${side}_wheel_joint" type="continuous">
+      <axis xyz="0 1 0" />
+      <parent link="base_link"/>
+      <child link="${side}_wheel_link"/>
+      <origin xyz="${pos_x} ${pos_y} ${pos_z}" rpy="0 0 0"/>
+    </joint>
+  </xacro:macro>
+</robot>

File: install/linorobot2_description/share/linorobot2_description/urdf/mech/wheel.urdf.xacro (robot description, xacro)
@@ -1 +1,45 @@
-/home/swarmmaster/thesis_ws/src/linorobot2/linorobot2_description/urdf/mech/wheel.urdf.xacro
+<?xml version="1.0"?>
+<robot xmlns:xacro="http://ros.org/wiki/xacro">
+  <xacro:macro name="wheel" params="side radius width pos_x pos_y pos_z mass">
+    <link name="${side}_wheel_link">
+      <visual>
+        <origin xyz="0 0 0" rpy="${pi/2} 0 0"/>
+        <geometry>
+          <cylinder radius="${radius}" length="${width}"/>
+        </geometry>
+        <material name="blue">
+            <color rgba="0.1764 0.4588 0.8509 1.0"/>
+        </material>
+      </visual>
+      <collision>
+        <origin xyz="0 0 0" rpy="${pi/2} 0 0"/>
+        <geometry>
+          <cylinder radius="${radius}" length="${width}"/>
+        </geometry>
+      </collision>
+      <inertial>
+        <origin xyz="0 0 0" rpy="0 0 0"/>
+        <mass value="${mass}"/>
+        <inertia ixx="${(2/5) * mass * (radius * radius)}" ixy="0" ixz="0"
+                 iyy="${(2/5) * mass * (radius * radius)}" iyz="0"
+                 izz="${(2/5) * mass * (radius * radius)}" />
+      </inertial>
+    </link>
+    <gazebo reference="${side}_wheel_link">
+      <visual>
+        <material>
+          <ambient>0.1764 0.4588 0.8509 1.0</ambient>
+          <diffuse>0.1764 0.4588 0.8509 1.0</diffuse>
+          <specular>0.1764 0.4588 0.8509 1.0</specular>
+          <emissive>0.0 0.0 0.0 0.0</emissive>
+        </material>
+      </visual>
+    </gazebo>
+    <joint name="${side}_wheel_joint" type="continuous">
+      <axis xyz="0 1 0" />
+      <parent link="base_link"/>
+      <child link="${side}_wheel_link"/>
+      <origin xyz="${pos_x} ${pos_y} ${pos_z}" rpy="0 0 0"/>
+    </joint>
+  </xacro:macro>
+</robot>

File: install/linorobot2_description/share/linorobot2_description/urdf/robots/2wd.urdf.xacro (robot description, xacro)
@@ -1 +1,67 @@
-/home/swarmmaster/thesis_ws/src/linorobot2/linorobot2_description/urdf/robots/2wd.urdf.xacro
+<?xml version="1.0"?>
+<robot name="linorobot2_2wd" xmlns:xacro="http://ros.org/wiki/xacro">
+  <xacro:include filename="$(find linorobot2_description)/urdf/2wd_properties.urdf.xacro" />
+  <xacro:include filename="$(find linorobot2_description)/urdf/mech/base.urdf.xacro" />
+  <xacro:include filename="$(find linorobot2_description)/urdf/mech/wheel.urdf.xacro" />
+  <xacro:include filename="$(find linorobot2_description)/urdf/mech/caster_wheel.urdf.xacro" />
+  <xacro:include filename="$(find linorobot2_description)/urdf/sensors/imu.urdf.xacro" />
+  <xacro:include filename="$(find linorobot2_description)/urdf/sensors/generic_laser.urdf.xacro" />
+  <xacro:include filename="$(find linorobot2_description)/urdf/sensors/depth_sensor.urdf.xacro" />
+  <xacro:include filename="$(find linorobot2_description)/urdf/controllers/diff_drive.urdf.xacro" />
+  <xacro:base
+    length="${base_length}"
+    width="${base_width}"
+    height="${base_height}"
+    mass="${base_mass}"
+    wheel_radius="${wheel_radius}"
+    wheel_pos_z="${wheel_pos_z}"
+/>
+  <xacro:wheel
+    side="left"
+    radius="${wheel_radius}"
+    width="${wheel_width}"
+    pos_x="${wheel_pos_x}"
+    pos_y="${wheel_pos_y}"
+    pos_z="${wheel_pos_z}"
+    mass="${wheel_mass}"
+  />
+  <xacro:wheel
+    side="right"
+    radius="${wheel_radius}"
+    width="${wheel_width}"
+    pos_x="${wheel_pos_x}"
+    pos_y="${-wheel_pos_y}"
+    pos_z="${wheel_pos_z}"
+    mass="${wheel_mass}"
+  />
+  <xacro:if value="${front_caster_wheel}">
+    <xacro:caster_wheel
+      side="front"
+      mass="0.01"
+      base_length="${base_length}"
+      wheel_radius="${wheel_radius}"
+      wheel_pos_z="${wheel_pos_z}"
+    />
+  </xacro:if>
+  <xacro:if value="${rear_caster_wheel}">
+    <xacro:caster_wheel
+      side="rear"
+      mass="0.01"
+      base_length="${base_length}"
+      wheel_radius="${wheel_radius}"
+      wheel_pos_z="${wheel_pos_z}"
+    />
+  </xacro:if>
+  <xacro:imu/>
+  <xacro:generic_laser>
+    <xacro:insert_block name="laser_pose" />
+  </xacro:generic_laser>
+  <xacro:depth_sensor>
+    <xacro:insert_block name="depth_sensor_pose" />
+  </xacro:depth_sensor>
+  <xacro:diff_drive_controller
+    wheel_separation="${wheel_pos_y * 2}"
+    wheel_radius="${wheel_radius}"
+    wheel_torque="${wheel_torque}"
+  />
+</robot>

File: install/linorobot2_description/share/linorobot2_description/urdf/robots/4wd.urdf.xacro (robot description, xacro)
@@ -1 +1,66 @@
-/home/swarmmaster/thesis_ws/src/linorobot2/linorobot2_description/urdf/robots/4wd.urdf.xacro
+<?xml version="1.0"?>
+<robot name="linorobot2_2wd" xmlns:xacro="http://ros.org/wiki/xacro">
+  <xacro:include filename="$(find linorobot2_description)/urdf/4wd_properties.urdf.xacro" />
+  <xacro:include filename="$(find linorobot2_description)/urdf/mech/base.urdf.xacro" />
+  <xacro:include filename="$(find linorobot2_description)/urdf/mech/wheel.urdf.xacro" />
+  <xacro:include filename="$(find linorobot2_description)/urdf/sensors/imu.urdf.xacro" />
+  <xacro:include filename="$(find linorobot2_description)/urdf/sensors/generic_laser.urdf.xacro" />
+  <xacro:include filename="$(find linorobot2_description)/urdf/sensors/depth_sensor.urdf.xacro" />
+  <xacro:include filename="$(find linorobot2_description)/urdf/controllers/skid_steer.urdf.xacro" />
+  <xacro:base
+    length="${base_length}"
+    width="${base_width}"
+    height="${base_height}"
+    mass="${base_mass}"
+    wheel_radius="${wheel_radius}"
+    wheel_pos_z="${wheel_pos_z}"
+/>
+  <xacro:wheel
+    side="front_left"
+    radius="${wheel_radius}"
+    width="${wheel_width}"
+    pos_x="${wheel_pos_x}"
+    pos_y="${wheel_pos_y}"
+    pos_z="${wheel_pos_z}"
+    mass="${wheel_mass}"
+  />
+  <xacro:wheel
+    side="front_right"
+    radius="${wheel_radius}"
+    width="${wheel_width}"
+    pos_x="${wheel_pos_x}"
+    pos_y="${-wheel_pos_y}"
+    pos_z="${wheel_pos_z}"
+    mass="${wheel_mass}"
+  />
+  <xacro:wheel
+    side="rear_left"
+    radius="${wheel_radius}"
+    width="${wheel_width}"
+    pos_x="${-wheel_pos_x}"
+    pos_y="${wheel_pos_y}"
+    pos_z="${wheel_pos_z}"
+    mass="${wheel_mass}"
+  />
+  <xacro:wheel
+    side="rear_right"
+    radius="${wheel_radius}"
+    width="${wheel_width}"
+    pos_x="${-wheel_pos_x}"
+    pos_y="${-wheel_pos_y}"
+    pos_z="${wheel_pos_z}"
+    mass="${wheel_mass}"
+  />
+  <xacro:imu/>
+  <xacro:generic_laser>
+    <xacro:insert_block name="laser_pose" />
+  </xacro:generic_laser>
+  <xacro:depth_sensor>
+    <xacro:insert_block name="depth_sensor_pose" />
+  </xacro:depth_sensor>
+  <xacro:diff_drive_controller
+    wheel_separation="${wheel_pos_y * 2}"
+    wheel_radius="${wheel_radius}"
+    wheel_torque="${wheel_torque}"
+  />
+</robot>
